File: ergogen/keyboards/macropad/config_4x5/pcbs/keyboard_numpad.kicad_pcb (KiCad board)
At the start: 2 copper layers, 50.6 x 95.9 mm, 63 parts

Commit message: Working ergogen-toolkit
Other:
- board size 50.6 x 95.9 mm -> 132.1 x 117.2 mm
Changed lines of the file:
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@@
         (pad 24 thru_hole circle (at 13.97 7.62 0) (size 1.7526 1.7526) (drill 1.0922) (layers *.Cu *.SilkS *.Mask) (net 45 "col_enc_bottom"))
       )
-  (gr_line (start 136.4 -104.3) (end 168.4 -104.3) (angle 90) (layer Edge.Cuts) (width 0.15))
+  (gr_line (start 47.625 -26.575000000000003) (end 90.3 -26.575000000000003) (angle 90) (layer Edge.Cuts) (width 0.15))
+(gr_line (start 93.3 -19.625000000000007) (end 93.3 -23.575000000000003) (angle 90) (layer Edge.Cuts) (width 0.15))
+(gr_arc (start 95.3 -19.625000000000007) (end 93.3 -19.625000000000007) (angle -90) (layer Edge.Cuts) (width 0.15))
+(gr_line (start 95.3 -17.625000000000007) (end 123.3 -17.625000000000007) (angle 90) (layer Edge.Cuts) (width 0.15))
+(gr_arc (start 123.3 -19.625000000000007) (end 123.3 -17.625000000000007) (angle -90) (layer Edge.Cuts) (width 0.15))
+(gr_line (start 125.3 -19.625000000000007) (end 125.29999999999998 -27.224305700000002) (angle 90) (layer Edge.Cuts) (width 0.15))
+(gr_arc (start 123.82499999999999 -28.575000000000003) (end 125.29999999999998 -27.224305700000002) (angle -42.48111359538382) (layer Edge.Cuts) (width 0.15))
+(gr_line (start 125.82499999999999 -28.575000000000003) (end 125.82499999999999 -123.825) (angle 90) (layer Edge.Cuts) (width 0.15))
+(gr_arc (start 123.82499999999999 -123.82499999999999) (end 125.82499999999999 -123.82499999999999) (angle -42.48111359538336) (layer Edge.Cuts) (width 0.15))
+(gr_line (start 125.29999999999998 -125.17569429999999) (end 125.3 -132.775) (angle 90) (layer Edge.Cuts) (width 0.15))
+(gr_arc (start 123.3 -132.775) (end 125.3 -132.775) (angle -90) (layer Edge.Cuts) (width 0.15))
+(gr_line (start 95.3 -134.775) (end 123.3 -134.775) (angle 90) (layer Edge.Cuts) (width 0.15))
+(gr_arc (start 95.3 -132.775) (end 95.3 -134.775) (angle -90) (layer Edge.Cuts) (width 0.15))
+(gr_line (start 93.3 -128.825) (end 93.3 -132.775) (angle 90) (layer Edge.Cuts) (width 0.15))
+(gr_line (start 47.625 -125.82499999999999) (end 90.3 -125.82499999999999) (angle 90) (layer Edge.Cuts) (width 0.15))
+(gr_arc (start 47.625 -123.825) (end 47.625 -125.825) (angle -90) (layer Edge.Cuts) (width 0.15))
+(gr_line (start 45.625 -28.575000000000003) (end 45.625 -123.825) (angle 90) (layer Edge.Cuts) (width 0.15))
+(gr_arc (start 47.625 -28.575000000000003) (end 45.625 -28.575000000000003) (angle -90) (layer Edge.Cuts) (width 0.15))
+(gr_line (start 100.3 -30.575000000000003) (end 118.3 -30.575000000000003) (angle 90) (layer Edge.Cuts) (width 0.15))
+(gr_line (start 121.3 -33.575) (end 121.3 -118.82499999999999) (angle 90) (layer Edge.Cuts) (width 0.15))
+(gr_line (start 100.3 -121.82499999999999) (end 118.3 -121.82499999999999) (angle 90) (layer Edge.Cuts) (width 0.15))
+(gr_line (start 97.3 -33.575) (end 97.3 -118.82499999999999) (angle 90) (layer Edge.Cuts) (width 0.15))
+(gr_line (start 136.4 -104.3) (end 168.4 -104.3) (angle 90) (layer Edge.Cuts) (width 0.15))
 (gr_arc (start 168.4 -106.3) (end 168.4 -104.3) (angle -90) (layer Edge.Cuts) (width 0.15))
 (gr_line (start 170.4 -106.3) (end 170.4 -122.3) (angle 90) (layer Edge.Cuts) (width 0.15))
@@
 (gr_line (start 141.4 -73.15) (end 141.4 -55.150000000000006) (angle 90) (layer Edge.Cuts) (width 0.15))
 (gr_arc (start 143.4 -55.150000000000006) (end 141.4 -55.150000000000006) (angle -90) (layer Edge.Cuts) (width 0.15))
+(gr_arc (start 90.3 -23.575000000000003) (end 93.3 -23.575000000000003) (angle -90) (layer Edge.Cuts) (width 0.15))
+(gr_arc (start 90.3 -128.825) (end 90.3 -125.82499999999999) (angle -90) (layer Edge.Cuts) (width 0.15))
+(gr_arc (start 118.3 -33.575) (end 118.3 -30.575000000000003) (angle -90) (layer Edge.Cuts) (width 0.15))
+(gr_arc (start 118.3 -118.82499999999999) (end 121.3 -118.82499999999999) (angle -90) (layer Edge.Cuts) (width 0.15))
+(gr_arc (start 100.3 -118.82499999999999) (end 100.3 -121.82499999999999) (angle -90) (layer Edge.Cuts) (width 0.15))
+(gr_arc (start 100.3 -33.575) (end 97.3 -33.575) (angle -90) (layer Edge.Cuts) (width 0.15))
 )

Commit message: More updates to the macropad
Other:
- board size 132.1 x 117.2 mm -> 169.1 x 108.2 mm
Changed lines of the file:
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@@
         (pad 24 thru_hole circle (at 13.97 7.62 0) (size 1.7526 1.7526) (drill 1.0922) (layers *.Cu *.SilkS *.Mask) (net 45 "col_enc_bottom"))
       )
-  (gr_line (start 47.625 -26.575000000000003) (end 90.3 -26.575000000000003) (angle 90) (layer Edge.Cuts) (width 0.15))
+  (gr_line (start 28.574999999999996 -26.575000000000003) (end 90.3 -26.575000000000003) (angle 90) (layer Edge.Cuts) (width 0.15))
 (gr_line (start 93.3 -19.625000000000007) (end 93.3 -23.575000000000003) (angle 90) (layer Edge.Cuts) (width 0.15))
 (gr_arc (start 95.3 -19.625000000000007) (end 93.3 -19.625000000000007) (angle -90) (layer Edge.Cuts) (width 0.15))
@@
 (gr_arc (start 123.82499999999999 -28.575000000000003) (end 125.29999999999998 -27.224305700000002) (angle -42.48111359538382) (layer Edge.Cuts) (width 0.15))
 (gr_line (start 125.82499999999999 -28.575000000000003) (end 125.82499999999999 -123.825) (angle 90) (layer Edge.Cuts) (width 0.15))
-(gr_arc (start 123.82499999999999 -123.82499999999999) (end 125.82499999999999 -123.82499999999999) (angle -42.48111359538336) (layer Edge.Cuts) (width 0.15))
-(gr_line (start 125.29999999999998 -125.17569429999999) (end 125.3 -132.775) (angle 90) (layer Edge.Cuts) (width 0.15))
-(gr_arc (start 123.3 -132.775) (end 125.3 -132.775) (angle -90) (layer Edge.Cuts) (width 0.15))
-(gr_line (start 95.3 -134.775) (end 123.3 -134.775) (angle 90) (layer Edge.Cuts) (width 0.15))
-(gr_arc (start 95.3 -132.775) (end 95.3 -134.775) (angle -90) (layer Edge.Cuts) (width 0.15))
-(gr_line (start 93.3 -128.825) (end 93.3 -132.775) (angle 90) (layer Edge.Cuts) (width 0.15))
-(gr_line (start 47.625 -125.82499999999999) (end 90.3 -125.82499999999999) (angle 90) (layer Edge.Cuts) (width 0.15))
-(gr_arc (start 47.625 -123.825) (end 47.625 -125.825) (angle -90) (layer Edge.Cuts) (width 0.15))
-(gr_line (start 45.625 -28.575000000000003) (end 45.625 -123.825) (angle 90) (layer Edge.Cuts) (width 0.15))
-(gr_arc (start 47.625 -28.575000000000003) (end 45.625 -28.575000000000003) (angle -90) (layer Edge.Cuts) (width 0.15))
+(gr_arc (start 123.82499999999999 -123.82499999999999) (end 125.82499999999999 -123.82499999999999) (angle -89.99999999999955) (layer Edge.Cuts) (width 0.15))
+(gr_line (start 28.574999999999996 -125.82499999999999) (end 123.82499999999999 -125.82499999999999) (angle 90) (layer Edge.Cuts) (width 0.15))
+(gr_arc (start 28.574999999999996 -123.825) (end 28.574999999999996 -125.825) (angle -42.48111359538382) (layer Edge.Cuts) (width 0.15))
+(gr_line (start 10.574999999999996 -125.3) (end 27.224305699999995 -125.3) (angle 90) (layer Edge.Cuts) (width 0.15))
+(gr_arc (start 10.574999999999996 -123.3) (end 10.574999999999996 -125.3) (angle -90) (layer Edge.Cuts) (width 0.15))
+(gr_line (start 8.574999999999996 -105.3) (end 8.574999999999996 -123.3) (angle 90) (layer Edge.Cuts) (width 0.15))
+(gr_arc (start 10.574999999999996 -105.3) (end 8.574999999999996 -105.3) (angle -90) (layer Edge.Cuts) (width 0.15))
+(gr_line (start 10.574999999999996 -103.3) (end 23.574999999999996 -103.3) (angle 90) (layer Edge.Cuts) (width 0.15))
+(gr_line (start 26.574999999999996 -28.575000000000003) (end 26.574999999999996 -100.3) (angle 90) (layer Edge.Cuts) (width 0.15))
+(gr_arc (start 28.574999999999996 -28.575000000000003) (end 26.574999999999996 -28.575000000000003) (angle -90) (layer Edge.Cuts) (width 0.15))
 (gr_line (start 100.3 -30.575000000000003) (end 118.3 -30.575000000000003) (angle 90) (layer Edge.Cuts) (width 0.15))
-(gr_line (start 121.3 -33.575) (end 121.3 -118.82499999999999) (angle 90) (layer Edge.Cuts) (width 0.15))
-(gr_line (start 100.3 -121.82499999999999) (end 118.3 -121.82499999999999) (angle 90) (layer Edge.Cuts) (width 0.15))
-(gr_line (start 97.3 -33.575) (end 97.3 -118.82499999999999) (angle 90) (layer Edge.Cuts) (width 0.15))
+(gr_line (start 121.3 -33.575) (end 121.3 -89.67500000000001) (angle 90) (layer Edge.Cuts) (width 0.15))
+(gr_line (start 100.3 -92.67500000000001) (end 118.3 -92.67500000000001) (angle 90) (layer Edge.Cuts) (width 0.15))
+(gr_line (start 97.3 -33.575) (end 97.3 -89.67500000000001) (angle 90) (layer Edge.Cuts) (width 0.15))
+(gr_line (start 30.574999999999996 -110.3) (end 30.574999999999996 -118.3) (angle 90) (layer Edge.Cuts) (width 0.15))
+(gr_line (start 33.574999999999996 -121.3) (end 79.675 -121.3) (angle 90) (layer Edge.Cuts) (width 0.15))
+(gr_line (start 82.675 -110.3) (end 82.675 -118.3) (angle 90) (layer Edge.Cuts) (width 0.15))
+(gr_line (start 33.574999999999996 -107.3) (end 79.675 -107.3) (angle 90) (layer Edge.Cuts) (width 0.15))
 (gr_line (start 136.4 -104.3) (end 168.4 -104.3) (angle 90) (layer Edge.Cuts) (width 0.15))
 (gr_arc (start 168.4 -106.3) (end 168.4 -104.3) (angle -90) (layer Edge.Cuts) (width 0.15))
@@
 (gr_arc (start 143.4 -55.150000000000006) (end 141.4 -55.150000000000006) (angle -90) (layer Edge.Cuts) (width 0.15))
 (gr_arc (start 90.3 -23.575000000000003) (end 93.3 -23.575000000000003) (angle -90) (layer Edge.Cuts) (width 0.15))
-(gr_arc (start 90.3 -128.825) (end 90.3 -125.82499999999999) (angle -90) (layer Edge.Cuts) (width 0.15))
+(gr_arc (start 23.574999999999996 -100.3) (end 26.574999999999996 -100.3) (angle -90) (layer Edge.Cuts) (width 0.15))
 (gr_arc (start 118.3 -33.575) (end 118.3 -30.575000000000003) (angle -90) (layer Edge.Cuts) (width 0.15))
-(gr_arc (start 118.3 -118.82499999999999) (end 121.3 -118.82499999999999) (angle -90) (layer Edge.Cuts) (width 0.15))
-(gr_arc (start 100.3 -118.82499999999999) (end 100.3 -121.82499999999999) (angle -90) (layer Edge.Cuts) (width 0.15))
+(gr_arc (start 118.3 -89.67500000000001) (end 121.3 -89.67500000000001) (angle -90) (layer Edge.Cuts) (width 0.15))
+(gr_arc (start 100.3 -89.67500000000001) (end 100.3 -92.67500000000001) (angle -90) (layer Edge.Cuts) (width 0.15))
 (gr_arc (start 100.3 -33.575) (end 97.3 -33.575) (angle -90) (layer Edge.Cuts) (width 0.15))
+(gr_arc (start 33.574999999999996 -118.3) (end 33.574999999999996 -121.3) (angle -90) (layer Edge.Cuts) (width 0.15))
+(gr_arc (start 79.675 -118.3) (end 82.675 -118.3) (angle -90) (layer Edge.Cuts) (width 0.15))
+(gr_arc (start 79.675 -110.3) (end 79.675 -107.3) (angle -90) (layer Edge.Cuts) (width 0.15))
+(gr_arc (start 33.574999999999996 -110.3) (end 30.574999999999996 -110.3) (angle -90) (layer Edge.Cuts) (width 0.15))
 )
